File: Connector.kicad_pcb (KiCad board)
At the start: 2 copper layers, 21.4 x 21.4 mm, 6 parts, among them J11 1pin_conn, J12 1pin_conn, J13 1pin_conn, J14 1pin_conn

Commit message: BOARD CORRECTIONS BASED ON PROTO TYPE
Parts:
- removed J13, J14: 1pin_conn, MyLib:Conn_1_Pin
Other:
- board text removed: "CKI"
- board text removed: "SDI"
Changed lines of the file:
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@@
   (general
     (thickness 1.6)
-    (drawings 29)
+    (drawings 27)
     (tracks 0)
     (zones 0)
-    (modules 6)
-    (nets 5)
+    (modules 4)
+    (nets 3)
   )
   (page A4)
@@
     (36 B.SilkS user)
     (37 F.SilkS user)
-    (38 B.Mask user)
-    (39 F.Mask user)
+    (38 B.Mask user hide)
+    (39 F.Mask user hide)
     (40 Dwgs.User user)
     (44 Edge.Cuts user)
@@
   (net 1 +5V)
   (net 2 GND)
-  (net 3 "Net-(J14-Pad1)")
-  (net 4 "Net-(J13-Pad1)")
   (net_class Default "This is the default net class."
     (clearance 0.2)
@@
     (add_net +5V)
     (add_net GND)
-    (add_net "Net-(J13-Pad1)")
-    (add_net "Net-(J14-Pad1)")
   )
   (module MyLib:Conn_1_Pin (layer F.Cu)
@@
     (pad 1 thru_hole circle (at -1 0) (size 0.8 0.8) (drill 0.4) (layers *.Cu *.Mask)
       (net 1 +5V))
-  )
-  (module MyLib:Conn_1_Pin (layer F.Cu)
-    (at 149.2 97.2)
-    (fp_text reference J13 (at -0.6 1.7) (layer F.SilkS) hide
-      (effects (font (size 1 1) (thickness 0.15)))
-    )
-    (fp_text value 1pin_conn (at 0 1.75) (layer F.Fab) hide
-      (effects (font (size 1 1) (thickness 0.15)))
-    )
-    (fp_line (start -1.75 0.72) (end -1.75 -0.75) (layer F.CrtYd) (width 0.12))
-    (fp_line (start 1.75 0.72) (end -1.75 0.72) (layer F.CrtYd) (width 0.12))
-    (fp_line (start 1.75 -0.76) (end 1.75 0.72) (layer F.CrtYd) (width 0.12))
-    (fp_line (start -1.75 -0.75) (end 1.75 -0.75) (layer F.CrtYd) (width 0.12))
-    (pad 1 smd rect (at 0 0) (size 3 1) (layers *.Mask B.Cu B.Paste)
-      (net 4 "Net-(J13-Pad1)"))
-    (pad 1 smd rect (at 0 0) (size 3 1) (layers F.Cu F.Paste F.Mask)
-      (net 4 "Net-(J13-Pad1)"))
-    (pad 1 thru_hole circle (at -1 0) (size 0.8 0.8) (drill 0.4) (layers *.Cu *.Mask)
-      (net 4 "Net-(J13-Pad1)"))
-  )
-  (module MyLib:Conn_1_Pin (layer F.Cu)
-    (at 152.6 97.2 180)
-    (fp_text reference J14 (at -0.7 -1.6) (layer F.SilkS) hide
-      (effects (font (size 1 1) (thickness 0.15)))
-    )
-    (fp_text value 1pin_conn (at 0 1.75) (layer F.Fab) hide
-      (effects (font (size 1 1) (thickness 0.15)))
-    )
-    (fp_line (start -1.75 0.72) (end -1.75 -0.75) (layer F.CrtYd) (width 0.12))
-    (fp_line (start 1.75 0.72) (end -1.75 0.72) (layer F.CrtYd) (width 0.12))
-    (fp_line (start 1.75 -0.76) (end 1.75 0.72) (layer F.CrtYd) (width 0.12))
-    (fp_line (start -1.75 -0.75) (end 1.75 -0.75) (layer F.CrtYd) (width 0.12))
-    (pad 1 smd rect (at 0 0 180) (size 3 1) (layers *.Mask B.Cu B.Paste)
-      (net 3 "Net-(J14-Pad1)"))
-    (pad 1 smd rect (at 0 0 180) (size 3 1) (layers F.Cu F.Paste F.Mask)
-      (net 3 "Net-(J14-Pad1)"))
-    (pad 1 thru_hole circle (at -1 0 180) (size 0.8 0.8) (drill 0.4) (layers *.Cu *.Mask)
-      (net 3 "Net-(J14-Pad1)"))
   )
   (dimension 21.410002 (width 0.15) (layer Dwgs.User)
@@
   (gr_arc (start 150.86 92.39) (end 159.32382 85.817096) (angle -104.3349919) (layer Edge.Cuts) (width 0.05))
   (target plus (at 140 103) (size 5) (width 0.05) (layer Edge.Cuts))
-  (gr_text CKI (at 148.6 98.6) (layer F.SilkS)
-    (effects (font (size 1 1) (thickness 0.15)))
-  )
-  (gr_text SDI (at 153.5 98.7) (layer F.SilkS)
-    (effects (font (size 1 1) (thickness 0.15)))
-  )
   (gr_text +5v (at 150.7 92.1) (layer F.SilkS)
     (effects (font (size 1 1) (thickness 0.15)))
@@
       )
     )
+  )
+  (zone (net 0) (net_name "") (layers F&B.Cu) (hatch edge 0.508)
+    (connect_pads (clearance 0))
+    (min_thickness 0.254)
+    (keepout (tracks allowed) (vias allowed) (copperpour not_allowed))
+    (fill (arc_segments 32) (thermal_gap 0.508) (thermal_bridge_width 0.508))
+    (polygon
+      (pts
+        (xy 154.2 98) (xy 147.5 98) (xy 147.5 95) (xy 154.2 95)
+      )
+    )
