File: Connector.kicad_pcb (KiCad board)
At the start: 2 copper layers, 21.4 x 21.4 mm, 4 parts, among them J11 1pin_conn, J12 1pin_conn

Commit message: Board Fixes fort bad footprint
Routing:
- net GND: vias 0 -> 1
Changed lines of the file:
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@@
   (general
     (thickness 1.6)
-    (drawings 27)
-    (tracks 0)
+    (drawings 29)
+    (tracks 1)
     (zones 0)
     (modules 4)
@@
       (net 1 +5V))
   )
+  (gr_poly (pts (xy 152.5 85.6) (xy 149.1 85.6) (xy 149.1 83.2) (xy 152.5 83.2)) (layer F.Mask) (width 0.1))
+  (gr_poly (pts (xy 152.5 85.6) (xy 149.1 85.6) (xy 149.1 83.2) (xy 152.5 83.2)) (layer B.Mask) (width 0.1))
   (dimension 21.410002 (width 0.15) (layer Dwgs.User)
     (gr_text "21.410 mm" (at 150.876611 76.545239 359.9732388) (layer Dwgs.User)
@@
     (effects (font (size 1 1) (thickness 0.15)))
   )
+  (via (at 150.8 84.4) (size 0.8) (drill 0.4) (layers F.Cu B.Cu) (net 2))
   (zone (net 1) (net_name +5V) (layer F.Cu) (hatch edge 0.508)
     (priority 4)
