File: Space fighter.kicad_pcb (KiCad board)
At the start: 2 copper layers, 73.3 x 42.5 mm, 9 parts, among them J2 6pin_conn

Commit message: more pictures for the doc's
Parts:
- removed C5, C6, C7, C8: .1uF, Capacitors_SMD:C_0603
- removed D5, D6, D7, D8: APA102-2020, MyLib:APA102-2020
- removed J2: 6pin_conn, MyLib:Connector
Routing:
- net Net-(D6-Pad2): track 89.3 -> 0.00 mm
- net Net-(D6-Pad3): track 87.0 -> 0.00 mm
- net Net-(D5-Pad5): track 83.6 -> 0.00 mm
- net Net-(D5-Pad4): track 83.6 -> 0.00 mm
- net Net-(D8-Pad2): track 16.4 -> 0.00 mm, vias 1 -> 0
- net Net-(D8-Pad3): track 14.2 -> 0.00 mm
- net GND: track 8.13 -> 0.00 mm, vias 7 -> 0
- net +5V: track 7.09 -> 0.00 mm, vias 4 -> 0
- net Net-(D5-Pad3): track 2.91 -> 0.00 mm, vias 1 -> 0
- net Net-(D5-Pad2): track 2.78 -> 0.00 mm, vias 1 -> 0
- net Net-(D7-Pad3): track 2.26 -> 0.00 mm, vias 1 -> 0
- net Net-(D7-Pad2): track 2.12 -> 0.00 mm, vias 1 -> 0
- removed copper zone on F.Cu, net +5V
- removed copper zone on B.Cu, net GND
Other:
- board outline removed
