File: Space fighter.sch (KiCad schematic (older format))
At the start: 28 parts, among them J10 6pin_conn, J11 1pin_conn, J12 1pin_conn, J13 1pin_conn, J14 1pin_conn, J2 6pin_conn, J7 6pin_conn, J8 6pin_conn, J9 6pin_conn, J99 Conn_01x06_Male

Commit message: Footprint was Jacked for LED - it's been fixed
foot print for led was incorrect.  It aslo seems that some pad resistors are needed
Parts:
- removed D2, D3, D4, D5, D6, D7, D8: APA102-2020, MyLib:APA102-2020, symbol LED:APA102-2020
- removed R1, R2: R_Small_US, Resistors_SMD:R_0805, symbol Device:R_Small_US
- added D2, D3, D4, D5, D6, D7, D8: APA102-2020, MyLib:APA102-2020_style_2, symbol MyComp:APA102-2020
- added R1, R2, R3, R4, R5, R6, R7, R8, R9: 33 ohm, Resistors_SMD:R_Array_Concave_2x0603, symbol Device:R_Pack02
- D1: footprint MyLib:APA102-2020 -> MyLib:APA102-2020_style_2; symbol LED:APA102-2020 -> MyComp:APA102-2020
Connections:
- net +5V: now also D1.7 (VDD), D2.1 (VDD), D2.7 (VDD), D3.1 (VDD), D3.7 (VDD), D4.1 (VDD), D4.7 (VDD), D5.1 (VDD), D5.7 (VDD), D6.1 (VDD), D6.7 (VDD), D7.1 (VDD), D7.7 (VDD), D8.1 (VDD), D8.7 (VDD)
- net GND: now also D1.8 (GND), D2.6 (GND), D2.8 (GND), D3.6 (GND), D3.8 (GND), D4.6 (GND), D4.8 (GND), D5.6 (GND), D5.8 (GND), D6.6 (GND), D6.8 (GND), D7.6 (GND), D7.8 (GND), D8.6 (GND), D8.8 (GND), R5.3 (R2.2), R5.4 (R1.2)
- net at D1.2 (CKO): now also R2.2 (R2.1)
- net at D1.3 (SDO): now also R2.1 (R1.1)
- net at D1.4 (SDI): now also R1.4 (R1.2); no longer J14.1
- net at D1.5 (CKI): now also R1.3 (R2.2); no longer J13.1
- net at J7.2: now also D4.2 (CKO)
- net at J7.1: now also D4.3 (SDO)
- net at J2.1: now also R6.2 (R2.1)
- net at J2.2: now also R6.1 (R1.1)
- net at J2.6: now also D8.2 (CKO)
- net at J2.5: now also D8.3 (SDO)
- net at J10.6: now also R5.1 (R1.1)
- net at J10.5: now also R5.2 (R2.1)
- new net: J13.1, R1.2 (R2.1)
- new net: J14.1, R1.1 (R1.1)
- new net: D2.5 (CKI), R2.3 (R2.2)
- new net: D2.4 (SDI), R2.4 (R1.2)
- new net: D2.2 (CKO), R3.2 (R2.1)
- new net: D2.3 (SDO), R3.1 (R1.1)
- new net: D3.5 (CKI), R3.3 (R2.2)
- new net: D3.4 (SDI), R3.4 (R1.2)
- new net: D3.2 (CKO), R4.2 (R2.1)
- new net: D3.3 (SDO), R4.1 (R1.1)
- new net: D4.5 (CKI), R4.3 (R2.2)
- new net: D4.4 (SDI), R4.4 (R1.2)
- new net: D5.2 (CKO), R7.1 (R1.1)
- new net: D5.3 (SDO), R7.2 (R2.1)
- new net: D5.4 (SDI), R6.3 (R2.2)
- new net: D5.5 (CKI), R6.4 (R1.2)
- new net: D6.4 (SDI), R7.3 (R2.2)
- new net: D6.5 (CKI), R7.4 (R1.2)
- new net: D6.2 (CKO), R8.1 (R1.1)
- new net: D6.3 (SDO), R8.2 (R2.1)
- new net: D7.4 (SDI), R8.3 (R2.2)
- new net: D7.5 (CKI), R8.4 (R1.2)
- new net: D7.2 (CKO), R9.1 (R1.1)
- new net: D7.3 (SDO), R9.2 (R2.1)
- new net: D8.4 (SDI), R9.3 (R2.2)
- new net: D8.5 (CKI), R9.4 (R1.2)
Other:
- moved on the sheet: C1, C2, C3, C4, C5, C6, C7, C8, J10A, J10B, J10C, J10D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
